File: 3_PCB/PCB_Projet/PCB_projet_V1/PCB_projet_V1.kicad_pcb (KiCad board)
At the start: 2 copper layers, 42 x 47.5 mm, 27 parts, among them U1 ADA4622-4ARZ, U2 ADA4622-4ARZ

Commit message: PCB erreurs
Parts:
- added J1: Conn_01x06_Pin, Connector_PinHeader_2.54mm:PinHeader_1x06_P2.54mm_Vertical, F.Cu at (75.8, 39.0)
- added J2: Conn_01x06_Pin, Connector_PinHeader_2.54mm:PinHeader_1x06_P2.54mm_Vertical, F.Cu at (84.9, 26.0)
- added J3: Conn_01x06_Pin, Connector_PinHeader_2.54mm:PinHeader_1x06_P2.54mm_Vertical, F.Cu at (104.8, 31.0)
- added J4: Conn_01x06_Pin, Connector_PinHeader_2.54mm:PinHeader_1x06_P2.54mm_Vertical, F.Cu at (84.8, 30.0)
Connections:
- A1 pad 1: unconnected-(A1-D1/TX-Pad1) -> Servomoteur T
- A1 pad 12: unconnected-(A1-D9-Pad12) -> LED GREEN
- A1 pad 13: unconnected-(A1-D10-Pad13) -> LED RED
- A1 pad 2: unconnected-(A1-D0/RX-Pad2) -> Servomoteur R
- A1 pad 30: unconnected-(A1-VIN-Pad30) -> +3.3V
- A1 pad 7: unconnected-(A1-D4-Pad7) -> OLED SDA
- A1 pad 8: unconnected-(A1-D5-Pad8) -> OLED SCL
Routing:
- net +5V: track 52.7 -> 81.8 mm, vias 2 -> 0
- net +3.3V: track 0.00 -> 26.7 mm
- net LED GREEN: track 0.00 -> 22.6 mm
- net LED RED: track 0.00 -> 21.4 mm
- net OLED SCL: track 0.00 -> 14.6 mm
- net OLED SDA: track 0.00 -> 13.7 mm
- net Servomoteur R: track 0.00 -> 6.92 mm
- net Servomoteur T: track 0.00 -> 6.92 mm
Other:
- board size 42 x 47.5 mm -> 50.5 x 60 mm
