File: 3_PCB/PCB_Projet/PCB_projet_V1/PCB_projet_V1.kicad_sch (KiCad schematic)
At the start: 33 parts, among them U1 ADA4622-4ARZ, U2 ADA4622-4ARZ

Commit message: PCB erreurs
Parts:
- removed GPIO3, GPIO4, GPIO5, GPIO6, GPIO7, GPIO8: Conn_01x01_Pin, Connector_PinHeader_2.54mm:PinHeader_1x01_P2.54mm_Vertical, symbol Connector:Conn_01x01_Pin
- added J1, J2, J3, J4: Conn_01x06_Pin, Connector_PinHeader_2.54mm:PinHeader_1x06_P2.54mm_Vertical, symbol Connector:Conn_01x06_Pin
Connections:
- net +5V: now also J2.1 (Pin_1), J2.2 (Pin_2), J2.3 (Pin_3), J2.4 (Pin_4), J2.5 (Pin_5), J2.6 (Pin_6)
- net GND: now also J3.1 (Pin_1), J3.2 (Pin_2), J3.3 (Pin_3), J3.4 (Pin_4), J3.5 (Pin_5), J3.6 (Pin_6)
- net LED GREEN: now also J1.5 (Pin_5)
- net LED RED: now also J1.6 (Pin_6)
- net OLED SCL: now also J1.4 (Pin_4)
- net OLED SDA: now also J1.3 (Pin_3)
- net Servomoteur R: now also J1.2 (Pin_2)
- net Servomoteur T: now also J1.1 (Pin_1)
- net +3.3V: now reaches A1.30 (VIN)
- net +3.3V: now also J4.1 (Pin_1), J4.2 (Pin_2), J4.3 (Pin_3), J4.4 (Pin_4), J4.5 (Pin_5), J4.6 (Pin_6)
Other:
- note added: "Composants"
- note removed: "Servomoteur"
